Commit message: Renomeia pacote adam para adam_urdf
Evita ambiguidade entre o nome do pacote ROS e o nome do robo "Adam".
Renomeacao completa, nao so a pasta:

- src/adam/ -> src/adam_urdf/ (git mv)
- package.xml: <name>adam</name> -> <name>adam_urdf</name>
- CMakeLists.txt: project(adam) -> project(adam_urdf)
- ~150 ocorrencias de package://adam/meshes/... -> package://adam_urdf/
  em adam.urdf, adam_fixed.urdf e adam.csv; adam.urdf.xacro regenerado
  via gen_xacro.py (nao editado a mao) a partir do adam_fixed.urdf
  corrigido
- get_package_share_directory('adam') / FindPackageShare('adam) -> 'adam_urdf'
  em display.launch.py, gazebo.launch.py, mock.launch.py (pacote adam_urdf),
  visualizar_marcha.launch.py (ax12_control) e demo.launch.py
  (adam_moveit_config)
- display.launch (ROS1 legado) tambem atualizado por consistencia

Nao alterado: MoveItConfigsBuilder("adam", package_name="adam_moveit_config")
em demo.launch.py/move_group.launch.py - esse "adam" e o nome do
robo/SRDF (adam.srdf), nao o nome do pacote URDF.

Validado com colcon build (ax12_control + adam_urdf + adam_moveit_config),
processamento do xacro + check_urdf (16 links) e resolucao dos meshes
via ros2 pkg prefix, antes de comitar.

Co-Authored-By: Claude Sonnet 4.6 <noreply@anthropic.com>

File: src/adam_urdf/urdf/adam.urdf (robot description, URDF)
Before this commit: robot adam, 17 links, 16 joints
Links:
- link base_link: geometry collision mesh filename=package://adam_urdf/meshes/base_link.STL; visual mesh filename=package://adam_urdf/meshes/base_link.STL
- link bd_antibraco: geometry collision mesh filename=package://adam_urdf/meshes/bd_antibraco.STL; visual mesh filename=package://adam_urdf/meshes/bd_antibraco.STL
- link bd_biceps: geometry collision mesh filename=package://adam_urdf/meshes/bd_biceps.STL; visual mesh filename=package://adam_urdf/meshes/bd_biceps.STL
- link bd_ombro: geometry collision mesh filename=package://adam_urdf/meshes/bd_ombro.STL; visual mesh filename=package://adam_urdf/meshes/bd_ombro.STL
- link be_antibraco: geometry collision mesh filename=package://adam_urdf/meshes/be_antibraco.STL; visual mesh filename=package://adam_urdf/meshes/be_antibraco.STL
- link be_biceps: geometry collision mesh filename=package://adam_urdf/meshes/be_biceps.STL; visual mesh filename=package://adam_urdf/meshes/be_biceps.STL
- link be_ombro: geometry collision mesh filename=package://adam_urdf/meshes/be_ombro.STL; visual mesh filename=package://adam_urdf/meshes/be_ombro.STL
- link pd_canela: geometry collision mesh filename=package://adam_urdf/meshes/pd_canela.STL; visual mesh filename=package://adam_urdf/meshes/pd_canela.STL
- link pd_coxa: geometry collision mesh filename=package://adam_urdf/meshes/pd_coxa.STL; visual mesh filename=package://adam_urdf/meshes/pd_coxa.STL
- link pd_pe: geometry collision mesh filename=package://adam_urdf/meshes/pd_pe.STL; visual mesh filename=package://adam_urdf/meshes/pd_pe.STL
- link pd_quadril: geometry collision mesh filename=package://adam_urdf/meshes/pd_quadril.STL; visual mesh filename=package://adam_urdf/meshes/pd_quadril.STL
- link pd_tornozelo: geometry collision mesh filename=package://adam_urdf/meshes/pd_tornozelo.STL; visual mesh filename=package://adam_urdf/meshes/pd_tornozelo.STL
- link pe_canela: geometry collision mesh filename=package://adam_urdf/meshes/pe_canela.STL; visual mesh filename=package://adam_urdf/meshes/pe_canela.STL
- link pe_coxa: geometry collision mesh filename=package://adam_urdf/meshes/pe_coxa.STL; visual mesh filename=package://adam_urdf/meshes/pe_coxa.STL
- link pe_pe: geometry collision mesh filename=package://adam_urdf/meshes/pe_pe.STL; visual mesh filename=package://adam_urdf/meshes/pe_pe.STL
- link pe_quadril: geometry collision mesh filename=package://adam_urdf/meshes/pe_quadril.STL; visual mesh filename=package://adam_urdf/meshes/pe_quadril.STL
- link pe_tornozelo: geometry collision mesh filename=package://adam_urdf/meshes/pe_tornozelo.STL; visual mesh filename=package://adam_urdf/meshes/pe_tornozelo.STL

File: src/adam_urdf/urdf/adam.urdf.xacro (robot description, xacro)
@@ -1,4 +1,7 @@
-<?xml version='1.0' encoding='utf-8'?>
-<robot name="adam">
+<?xml version="1.0" encoding="utf-8"?>
+<!-- GERADO por gen_xacro.py a partir de adam.urdf. Nao editar a mao;
+     edite gen_xacro.py ou adam.urdf e rode o script de novo. -->
+<robot name="adam" xmlns:xacro="http://www.ros.org/wiki/xacro">
+  <xacro:arg name="use_mock_hardware" default="true"/>
   <link name="base_link">
     <inertial>
@@ -10,5 +13,5 @@
       <origin xyz="0 0 0" rpy="0 0 0" />
       <geometry>
-        <mesh filename="package://adam/meshes/base_link.STL" />
+        <mesh filename="package://adam_urdf/meshes/base_link.STL" />
       </geometry>
       <material name="">
@@ -19,5 +22,5 @@
       <origin xyz="0 0 0" rpy="0 0 0" />
       <geometry>
-        <mesh filename="package://adam/meshes/base_link.STL" />
+        <mesh filename="package://adam_urdf/meshes/base_link.STL" />
       </geometry>
     </collision>
@@ -32,5 +35,5 @@
       <origin xyz="0.03625008 -0.01049992 -0.02299991" rpy="-2.35619449 -1.57079113 -2.35619449" />
       <geometry>
-        <mesh filename="package://adam/meshes/pe_quadril.STL" />
+        <mesh filename="package://adam_urdf/meshes/pe_quadril.STL" />
       </geometry>
       <material name="">
@@ -41,5 +44,5 @@
       <origin xyz="0.03625008 -0.01049992 -0.02299991" rpy="-2.35619449 -1.57079113 -2.35619449" />
       <geometry>
-        <mesh filename="package://adam/meshes/pe_quadril.STL" />
+        <mesh filename="package://adam_urdf/meshes/pe_quadril.STL" />
       </geometry>
     </collision>
@@ -61,5 +64,5 @@
       <origin xyz="0.05790780 0.00175479 0.03045030" rpy="-1.57079265 0.00000735 -1.57079265" />
       <geometry>
-        <mesh filename="package://adam/meshes/pe_coxa.STL" />
+        <mesh filename="package://adam_urdf/meshes/pe_coxa.STL" />
       </geometry>
       <material name="">
@@ -70,5 +73,5 @@
       <origin xyz="0.05790780 0.00175479 0.03045030" rpy="-1.57079265 0.00000735 -1.57079265" />
       <geometry>
-        <mesh filename="package://adam/meshes/pe_coxa.STL" />
+        <mesh filename="package://adam_urdf/meshes/pe_coxa.STL" />
       </geometry>
     </collision>
@@ -79,5 +82,5 @@
     <child link="pe_coxa" />
     <axis xyz="0 0 1" />
-    <limit lower="-2.618" upper="2.618" effort="1.5" velocity="11.9" />
+    <limit lower="-2.6180" upper="2.6180" effort="1.5" velocity="6.0" />
   </joint>
   <link name="pe_canela">
@@ -90,5 +93,5 @@
       <origin xyz="-0.01394569 -0.13230775 0.03045030" rpy="-1.57079265 0.00000735 -3.14159265" />
       <geometry>
-        <mesh filename="package://adam/meshes/pe_canela.STL" />
+        <mesh filename="package://adam_urdf/meshes/pe_canela.STL" />
       </geometry>
       <material name="">
@@ -99,5 +102,5 @@
       <origin xyz="-0.01394569 -0.13230775 0.03045030" rpy="-1.57079265 0.00000735 -3.14159265" />
       <geometry>
-        <mesh filename="package://adam/meshes/pe_canela.STL" />
+        <mesh filename="package://adam_urdf/meshes/pe_canela.STL" />
       </geometry>
     </collision>
@@ -108,5 +111,5 @@
     <child link="pe_canela" />
     <axis xyz="0 0 1" />
-    <limit lower="-2.618" upper="2.618" effort="1.5" velocity="11.9" />
+    <limit lower="-2.6180" upper="0.0000" effort="1.5" velocity="6.0" />
   </joint>
   <link name="pe_tornozelo">
@@ -119,5 +122,5 @@
       <origin xyz="-0.20754875 0.00075345 0.03045030" rpy="-1.57079265 0.00000735 1.57079265" />
       <geometry>
-        <mesh filename="package://adam/meshes/pe_tornozelo.STL" />
+        <mesh filename="package://adam_urdf/meshes/pe_tornozelo.STL" />
       </geometry>
       <material name="">
@@ -128,5 +131,5 @@
       <origin xyz="-0.20754875 0.00075345 0.03045030" rpy="-1.57079265 0.00000735 1.57079265" />
       <geometry>
-        <mesh filename="package://adam/meshes/pe_tornozelo.STL" />
+        <mesh filename="package://adam_urdf/meshes/pe_tornozelo.STL" />
       </geometry>
     </collision>
@@ -137,5 +140,5 @@
     <child link="pe_tornozelo" />
     <axis xyz="0 0 1" />
-    <limit lower="-2.618" upper="2.618" effort="1.5" velocity="11.9" />
+    <limit lower="-0.5585" upper="1.4661" effort="1.5" velocity="6.0" />
   </joint>
   <link name="pe_pe">
@@ -148,5 +151,5 @@
       <origin xyz="-0.20764875 -0.05165039 0.02455327" rpy="-0.78539449 -1.57079113 0.78539816" />
       <geometry>
-        <mesh filename="package://adam/meshes/pe_pe.STL" />
+        <mesh filename="package://adam_urdf/meshes/pe_pe.STL" />
       </geometry>
       <material name="">
@@ -157,5 +160,5 @@
       <origin xyz="-0.20764875 -0.05165039 0.02455327" rpy="-0.78539449 -1.57079113 0.78539816" />
       <geometry>
-        <mesh filename="package://adam/meshes/pe_pe.STL" />
+        <mesh filename="package://adam_urdf/meshes/pe_pe.STL" />
       </geometry>
     </collision>
@@ -166,5 +169,5 @@
     <child link="pe_pe" />
     <axis xyz="0 0 1" />
-    <limit lower="-2.618" upper="2.618" effort="1.5" velocity="11.9" />
+    <limit lower="-0.5934" upper="0.8727" effort="1.5" velocity="6.0" />
   </joint>
   <link name="pd_quadril">
@@ -177,5 +180,5 @@
       <origin xyz="0.03625008 0.01049992 -0.02299991" rpy="2.35619449 -1.57079113 2.35619449" />
       <geometry>
-        <mesh filename="package://adam/meshes/pd_quadril.STL" />
+        <mesh filename="package://adam_urdf/meshes/pd_quadril.STL" />
       </geometry>
       <material name="">
@@ -186,5 +189,5 @@
       <origin xyz="0.03625008 0.01049992 -0.02299991" rpy="2.35619449 -1.57079113 2.35619449" />
       <geometry>
-        <mesh filename="package://adam/meshes/pd_quadril.STL" />
+        <mesh filename="package://adam_urdf/meshes/pd_quadril.STL" />
       </geometry>
     </collision>
@@ -206,5 +209,5 @@
       <origin xyz="0.05790780 -0.00175479 0.03045030" rpy="1.57079265 0.00000735 1.57079265" />
       <geometry>
-        <mesh filename="package://adam/meshes/pd_coxa.STL" />
+        <mesh filename="package://adam_urdf/meshes/pd_coxa.STL" />
       </geometry>
       <material name="">
@@ -215,5 +218,5 @@
       <origin xyz="0.05790780 -0.00175479 0.03045030" rpy="1.57079265 0.00000735 1.57079265" />
       <geometry>
-        <mesh filename="package://adam/meshes/pd_coxa.STL" />
+        <mesh filename="package://adam_urdf/meshes/pd_coxa.STL" />
       </geometry>
     </collision>
@@ -224,5 +227,5 @@
     <child link="pd_coxa" />
     <axis xyz="0 0 1" />
-    <limit lower="-2.618" upper="2.618" effort="1.5" velocity="11.9" />
+    <limit lower="-2.6180" upper="2.6180" effort="1.5" velocity="6.0" />
   </joint>
   <link name="pd_canela">
@@ -235,5 +238,5 @@
       <origin xyz="-0.01394569 0.13230775 0.03045030" rpy="1.57079265 0.00000735 3.14159265" />
       <geometry>
-        <mesh filename="package://adam/meshes/pd_canela.STL" />
+        <mesh filename="package://adam_urdf/meshes/pd_canela.STL" />
       </geometry>
       <material name="">
@@ -244,5 +247,5 @@
       <origin xyz="-0.01394569 0.13230775 0.03045030" rpy="1.57079265 0.00000735 3.14159265" />
       <geometry>
-        <mesh filename="package://adam/meshes/pd_canela.STL" />
+        <mesh filename="package://adam_urdf/meshes/pd_canela.STL" />
       </geometry>
     </collision>
@@ -253,5 +256,5 @@
     <child link="pd_canela" />
     <axis xyz="0 0 1" />
-    <limit lower="-2.618" upper="2.618" effort="1.5" velocity="11.9" />
+    <limit lower="0.0000" upper="2.6180" effort="1.5" velocity="6.0" />
   </joint>
   <link name="pd_tornozelo">
@@ -264,5 +267,5 @@
       <origin xyz="-0.20754875 -0.00075345 0.03045030" rpy="1.57079265 0.00000735 -1.57079265" />
       <geometry>
-        <mesh filename="package://adam/meshes/pd_tornozelo.STL" />
+        <mesh filename="package://adam_urdf/meshes/pd_tornozelo.STL" />
       </geometry>
       <material name="">
@@ -273,5 +276,5 @@
       <origin xyz="-0.20754875 -0.00075345 0.03045030" rpy="1.57079265 0.00000735 -1.57079265" />
       <geometry>
-        <mesh filename="package://adam/meshes/pd_tornozelo.STL" />
+        <mesh filename="package://adam_urdf/meshes/pd_tornozelo.STL" />
       </geometry>
     </collision>
@@ -282,5 +285,5 @@
     <child link="pd_tornozelo" />
     <axis xyz="0 0 1" />
-    <limit lower="-2.618" upper="2.618" effort="1.5" velocity="11.9" />
+    <limit lower="-1.4661" upper="0.5585" effort="1.5" velocity="6.0" />
   </joint>
   <link name="pd_pe">
@@ -293,5 +296,5 @@
       <origin xyz="-0.20764875 0.05145040 0.02545327" rpy="0.78539449 -1.57079113 -0.78539816" />
       <geometry>
-        <mesh filename="package://adam/meshes/pd_pe.STL" />
+        <mesh filename="package://adam_urdf/meshes/pd_pe.STL" />
       </geometry>
       <material name="">
@@ -302,5 +305,5 @@
       <origin xyz="-0.20764875 0.05145040 0.02545327" rpy="0.78539449 -1.57079113 -0.78539816" />
       <geometry>
-        <mesh filename="package://adam/meshes/pd_pe.STL" />
+        <mesh filename="package://adam_urdf/meshes/pd_pe.STL" />
       </geometry>
     </collision>
@@ -311,5 +314,5 @@
     <child link="pd_pe" />
     <axis xyz="0 0 1" />
-    <limit lower="-2.618" upper="2.618" effort="1.5" velocity="11.9" />
+    <limit lower="-0.8727" upper="0.5934" effort="1.5" velocity="6.0" />
   </joint>
   <link name="be_ombro">
@@ -322,5 +325,5 @@
       <origin xyz="-0.17620805 0.00549938 -0.08799998" rpy="1.57079647 -0.00000367 1.53300000" />
       <geometry>
-        <mesh filename="package://adam/meshes/be_ombro.STL" />
+        <mesh filename="package://adam_urdf/meshes/be_ombro.STL" />
       </geometry>
       <material name="">
@@ -331,5 +334,5 @@
       <origin xyz="-0.17620805 0.00549938 -0.08799998" rpy="1.57079647 -0.00000367 1.53300000" />
       <geometry>
-        <mesh filename="package://adam/meshes/be_ombro.STL" />
+        <mesh filename="package://adam_urdf/meshes/be_ombro.STL" />
       </geometry>
     </collision>
@@ -351,5 +354,5 @@
       <origin xyz="-0.15828976 0.11100006 -0.02216938" rpy="-0.19251951 -1.57075794 -2.94907300" />
       <geometry>
-        <mesh filename="package://adam/meshes/be_biceps.STL" />
+        <mesh filename="package://adam_urdf/meshes/be_biceps.STL" />
       </geometry>
       <material name="">
@@ -360,5 +363,5 @@
       <origin xyz="-0.15828976 0.11100006 -0.02216938" rpy="-0.19251951 -1.57075794 -2.94907300" />
       <geometry>
-        <mesh filename="package://adam/meshes/be_biceps.STL" />
+        <mesh filename="package://adam_urdf/meshes/be_biceps.STL" />
       </geometry>
     </collision>
@@ -380,5 +383,5 @@
       <origin xyz="-0.01936902 0.09838934 -0.13200042" rpy="1.57079279 -0.00000734 0.00003400" />
       <geometry>
-        <mesh filename="package://adam/meshes/be_antibraco.STL" />
+        <mesh filename="package://adam_urdf/meshes/be_antibraco.STL" />
       </geometry>
       <material name="">
@@ -389,5 +392,5 @@
       <origin xyz="-0.01936902 0.09838934 -0.13200042" rpy="1.57079279 -0.00000734 0.00003400" />
       <geometry>
-        <mesh filename="package://adam/meshes/be_antibraco.STL" />
+        <mesh filename="package://adam_urdf/meshes/be_antibraco.STL" />
       </geometry>
     </collision>
@@ -409,5 +412,5 @@
       <origin xyz="-0.17620805 -0.00549938 -0.08799998" rpy="-1.57079647 -0.00000367 -1.53300000" />
       <geometry>
-        <mesh filename="package://adam/meshes/bd_ombro.STL" />
+        <mesh filename="package://adam_urdf/meshes/bd_ombro.STL" />
       </geometry>
       <material name="">
@@ -418,5 +421,5 @@
       <origin xyz="-0.17620805 -0.00549938 -0.08799998" rpy="-1.57079647 -0.00000367 -1.53300000" />
       <geometry>
-        <mesh filename="package://adam/meshes/bd_ombro.STL" />
+        <mesh filename="package://adam_urdf/meshes/bd_ombro.STL" />
       </geometry>
     </collision>
@@ -438,5 +441,5 @@
       <origin xyz="-0.15828976 -0.11100006 -0.02216938" rpy="0.19251951 -1.57075794 2.94907300" />
       <geometry>
-        <mesh filename="package://adam/meshes/bd_biceps.STL" />
+        <mesh filename="package://adam_urdf/meshes/bd_biceps.STL" />
       </geometry>
       <material name="">
@@ -447,5 +450,5 @@
       <origin xyz="-0.15828976 -0.11100006 -0.02216938" rpy="0.19251951 -1.57075794 2.94907300" />
       <geometry>
-        <mesh filename="package://adam/meshes/bd_biceps.STL" />
+        <mesh filename="package://adam_urdf/meshes/bd_biceps.STL" />
       </geometry>
     </collision>
@@ -467,5 +470,5 @@
       <origin xyz="-0.01936974 -0.09839022 -0.13199967" rpy="-1.57080049 -0.00000734 -0.00004135" />
       <geometry>
-        <mesh filename="package://adam/meshes/bd_antibraco.STL" />
+        <mesh filename="package://adam_urdf/meshes/bd_antibraco.STL" />
       </geometry>
       <material name="">
@@ -476,5 +479,5 @@
       <origin xyz="-0.01936974 -0.09839022 -0.13199967" rpy="-1.57080049 -0.00000734 -0.00004135" />
       <geometry>
-        <mesh filename="package://adam/meshes/bd_antibraco.STL" />
+        <mesh filename="package://adam_urdf/meshes/bd_antibraco.STL" />
       </geometry>
     </collision>
@@ -487,3 +490,6 @@
     <limit lower="-2.618" upper="2.618" effort="1.5" velocity="11.9" />
   </joint>
+  <xacro:include filename="adam.ros2_control.xacro"/>
+  <xacro:adam_ros2_control name="AdamSystem"
+      use_mock_hardware="$(arg use_mock_hardware)"/>
 </robot>

File: src/adam_urdf/urdf/adam_fixed.urdf (robot description, URDF)
Before this commit: robot adam, 17 links, 16 joints
Links:
- link base_link: geometry collision mesh filename=package://adam_urdf/meshes/base_link.STL; visual mesh filename=package://adam_urdf/meshes/base_link.STL
- link bd_antibraco: geometry collision mesh filename=package://adam_urdf/meshes/bd_antibraco.STL; visual mesh filename=package://adam_urdf/meshes/bd_antibraco.STL
- link bd_biceps: geometry collision mesh filename=package://adam_urdf/meshes/bd_biceps.STL; visual mesh filename=package://adam_urdf/meshes/bd_biceps.STL
- link bd_ombro: geometry collision mesh filename=package://adam_urdf/meshes/bd_ombro.STL; visual mesh filename=package://adam_urdf/meshes/bd_ombro.STL
- link be_antibraco: geometry collision mesh filename=package://adam_urdf/meshes/be_antibraco.STL; visual mesh filename=package://adam_urdf/meshes/be_antibraco.STL
- link be_biceps: geometry collision mesh filename=package://adam_urdf/meshes/be_biceps.STL; visual mesh filename=package://adam_urdf/meshes/be_biceps.STL
- link be_ombro: geometry collision mesh filename=package://adam_urdf/meshes/be_ombro.STL; visual mesh filename=package://adam_urdf/meshes/be_ombro.STL
- link pd_canela: geometry collision mesh filename=package://adam_urdf/meshes/pd_canela.STL; visual mesh filename=package://adam_urdf/meshes/pd_canela.STL
- link pd_coxa: geometry collision mesh filename=package://adam_urdf/meshes/pd_coxa.STL; visual mesh filename=package://adam_urdf/meshes/pd_coxa.STL
- link pd_pe: geometry collision mesh filename=package://adam_urdf/meshes/pd_pe.STL; visual mesh filename=package://adam_urdf/meshes/pd_pe.STL
- link pd_quadril: geometry collision mesh filename=package://adam_urdf/meshes/pd_quadril.STL; visual mesh filename=package://adam_urdf/meshes/pd_quadril.STL
- link pd_tornozelo: geometry collision mesh filename=package://adam_urdf/meshes/pd_tornozelo.STL; visual mesh filename=package://adam_urdf/meshes/pd_tornozelo.STL
- link pe_canela: geometry collision mesh filename=package://adam_urdf/meshes/pe_canela.STL; visual mesh filename=package://adam_urdf/meshes/pe_canela.STL
- link pe_coxa: geometry collision mesh filename=package://adam_urdf/meshes/pe_coxa.STL; visual mesh filename=package://adam_urdf/meshes/pe_coxa.STL
- link pe_pe: geometry collision mesh filename=package://adam_urdf/meshes/pe_pe.STL; visual mesh filename=package://adam_urdf/meshes/pe_pe.STL
- link pe_quadril: geometry collision mesh filename=package://adam_urdf/meshes/pe_quadril.STL; visual mesh filename=package://adam_urdf/meshes/pe_quadril.STL
- link pe_tornozelo: geometry collision mesh filename=package://adam_urdf/meshes/pe_tornozelo.STL; visual mesh filename=package://adam_urdf/meshes/pe_tornozelo.STL
Joints:
- joint pd_picht_joelho_5: limit lower=0.0000 upper=2.6180 effort=1.5 velocity=6.0 -> lower=-2.618 upper=2.618 effort=1.5 velocity=11.9
- joint pd_picht_quadril_7: limit lower=-2.6180 upper=2.6180 effort=1.5 velocity=6.0 -> lower=-2.618 upper=2.618 effort=1.5 velocity=11.9
- joint pd_picht_tornozelo_3: limit lower=-1.4661 upper=0.5585 effort=1.5 velocity=6.0 -> lower=-2.618 upper=2.618 effort=1.5 velocity=11.9
- joint pd_roll_tornozelo_1: limit lower=-0.8727 upper=0.5934 effort=1.5 velocity=6.0 -> lower=-2.618 upper=2.618 effort=1.5 velocity=11.9
- joint pe_pich_quadril_8: limit lower=-2.6180 upper=2.6180 effort=1.5 velocity=6.0 -> lower=-2.618 upper=2.618 effort=1.5 velocity=11.9
- joint pe_picht_joelho_6: limit lower=-2.6180 upper=0.0000 effort=1.5 velocity=6.0 -> lower=-2.618 upper=2.618 effort=1.5 velocity=11.9
- joint pe_picht_tornozelo_4: limit lower=-0.5585 upper=1.4661 effort=1.5 velocity=6.0 -> lower=-2.618 upper=2.618 effort=1.5 velocity=11.9
- joint pe_roll_tornozelo_2: limit lower=-0.5934 upper=0.8727 effort=1.5 velocity=6.0 -> lower=-2.618 upper=2.618 effort=1.5 velocity=11.9
