Commit message: limpeza 2: reorganiza pacotes no padrao ROS 2
Renomeia adam_urdf para adam_description (_description e o sufixo
padrao para um pacote so de URDF/malhas) e cria adam_bringup, para
onde vao config/ros2_controllers.yaml e launch/mock.launch.py. Subir
controller_manager nao e papel de um pacote _description, que volta a
ser dado puro do modelo.

Move gen_xacro.py e fix_urdf_origins.py para adam_description/scripts/
(estavam soltos em urdf/ e na raiz do pacote); ambos passam a resolver
caminhos relativos ao proprio arquivo. Remove export.log, 2259 linhas
de log bruto do plugin SW2URDF.

Corrige tambem: ax12_control/package.xml nao declarava dependencia do
pacote de descricao, apesar dos launch carregarem o URDF dele; e o
package.xml do adam_description tinha autor/maintainer TODO e licenca
BSD (o repositorio e MIT), sobras do exportador SolidWorks.

Validado: colcon build limpo nos 3 pacotes, os 7 launch files carregam
via --show-args, e gen_xacro.py regenera o adam.urdf.xacro identico.

Co-Authored-By: Claude Opus 5 <noreply@anthropic.com>

File: src/adam_description/urdf/adam.urdf (robot description, URDF)
Before this commit: robot adam, 17 links, 16 joints
Links:
- link base_link: geometry collision mesh filename=package://adam_description/meshes/base_link.STL; visual mesh filename=package://adam_description/meshes/base_link.STL
- link bd_antibraco: geometry collision mesh filename=package://adam_description/meshes/bd_antibraco.STL; visual mesh filename=package://adam_description/meshes/bd_antibraco.STL
- link bd_biceps: geometry collision mesh filename=package://adam_description/meshes/bd_biceps.STL; visual mesh filename=package://adam_description/meshes/bd_biceps.STL
- link bd_ombro: geometry collision mesh filename=package://adam_description/meshes/bd_ombro.STL; visual mesh filename=package://adam_description/meshes/bd_ombro.STL
- link be_antibraco: geometry collision mesh filename=package://adam_description/meshes/be_antibraco.STL; visual mesh filename=package://adam_description/meshes/be_antibraco.STL
- link be_biceps: geometry collision mesh filename=package://adam_description/meshes/be_biceps.STL; visual mesh filename=package://adam_description/meshes/be_biceps.STL
- link be_ombro: geometry collision mesh filename=package://adam_description/meshes/be_ombro.STL; visual mesh filename=package://adam_description/meshes/be_ombro.STL
- link pd_canela: geometry collision mesh filename=package://adam_description/meshes/pd_canela.STL; visual mesh filename=package://adam_description/meshes/pd_canela.STL
- link pd_coxa: geometry collision mesh filename=package://adam_description/meshes/pd_coxa.STL; visual mesh filename=package://adam_description/meshes/pd_coxa.STL
- link pd_pe: geometry collision mesh filename=package://adam_description/meshes/pd_pe.STL; visual mesh filename=package://adam_description/meshes/pd_pe.STL
- link pd_quadril: geometry collision mesh filename=package://adam_description/meshes/pd_quadril.STL; visual mesh filename=package://adam_description/meshes/pd_quadril.STL
- link pd_tornozelo: geometry collision mesh filename=package://adam_description/meshes/pd_tornozelo.STL; visual mesh filename=package://adam_description/meshes/pd_tornozelo.STL
- link pe_canela: geometry collision mesh filename=package://adam_description/meshes/pe_canela.STL; visual mesh filename=package://adam_description/meshes/pe_canela.STL
- link pe_coxa: geometry collision mesh filename=package://adam_description/meshes/pe_coxa.STL; visual mesh filename=package://adam_description/meshes/pe_coxa.STL
- link pe_pe: geometry collision mesh filename=package://adam_description/meshes/pe_pe.STL; visual mesh filename=package://adam_description/meshes/pe_pe.STL
- link pe_quadril: geometry collision mesh filename=package://adam_description/meshes/pe_quadril.STL; visual mesh filename=package://adam_description/meshes/pe_quadril.STL
- link pe_tornozelo: geometry collision mesh filename=package://adam_description/meshes/pe_tornozelo.STL; visual mesh filename=package://adam_description/meshes/pe_tornozelo.STL

File: src/adam_description/urdf/adam.urdf.xacro (robot description, xacro)
@@ -13,5 +13,5 @@
       <origin xyz="0 0 0" rpy="0 0 0" />
       <geometry>
-        <mesh filename="package://adam_urdf/meshes/base_link.STL" />
+        <mesh filename="package://adam_description/meshes/base_link.STL" />
       </geometry>
       <material name="">
@@ -22,5 +22,5 @@
       <origin xyz="0 0 0" rpy="0 0 0" />
       <geometry>
-        <mesh filename="package://adam_urdf/meshes/base_link.STL" />
+        <mesh filename="package://adam_description/meshes/base_link.STL" />
       </geometry>
     </collision>
@@ -35,5 +35,5 @@
       <origin xyz="0.03625008 -0.01049992 -0.02299991" rpy="-2.35619449 -1.57079113 -2.35619449" />
       <geometry>
-        <mesh filename="package://adam_urdf/meshes/pe_quadril.STL" />
+        <mesh filename="package://adam_description/meshes/pe_quadril.STL" />
       </geometry>
       <material name="">
@@ -44,5 +44,5 @@
       <origin xyz="0.03625008 -0.01049992 -0.02299991" rpy="-2.35619449 -1.57079113 -2.35619449" />
       <geometry>
-        <mesh filename="package://adam_urdf/meshes/pe_quadril.STL" />
+        <mesh filename="package://adam_description/meshes/pe_quadril.STL" />
       </geometry>
     </collision>
@@ -64,5 +64,5 @@
       <origin xyz="0.05790780 0.00175479 0.03045030" rpy="-1.57079265 0.00000735 -1.57079265" />
       <geometry>
-        <mesh filename="package://adam_urdf/meshes/pe_coxa.STL" />
+        <mesh filename="package://adam_description/meshes/pe_coxa.STL" />
       </geometry>
       <material name="">
@@ -73,5 +73,5 @@
       <origin xyz="0.05790780 0.00175479 0.03045030" rpy="-1.57079265 0.00000735 -1.57079265" />
       <geometry>
-        <mesh filename="package://adam_urdf/meshes/pe_coxa.STL" />
+        <mesh filename="package://adam_description/meshes/pe_coxa.STL" />
       </geometry>
     </collision>
@@ -93,5 +93,5 @@
       <origin xyz="-0.01394569 -0.13230775 0.03045030" rpy="-1.57079265 0.00000735 -3.14159265" />
       <geometry>
-        <mesh filename="package://adam_urdf/meshes/pe_canela.STL" />
+        <mesh filename="package://adam_description/meshes/pe_canela.STL" />
       </geometry>
       <material name="">
@@ -102,5 +102,5 @@
       <origin xyz="-0.01394569 -0.13230775 0.03045030" rpy="-1.57079265 0.00000735 -3.14159265" />
       <geometry>
-        <mesh filename="package://adam_urdf/meshes/pe_canela.STL" />
+        <mesh filename="package://adam_description/meshes/pe_canela.STL" />
       </geometry>
     </collision>
@@ -122,5 +122,5 @@
       <origin xyz="-0.20754875 0.00075345 0.03045030" rpy="-1.57079265 0.00000735 1.57079265" />
       <geometry>
-        <mesh filename="package://adam_urdf/meshes/pe_tornozelo.STL" />
+        <mesh filename="package://adam_description/meshes/pe_tornozelo.STL" />
       </geometry>
       <material name="">
@@ -131,5 +131,5 @@
       <origin xyz="-0.20754875 0.00075345 0.03045030" rpy="-1.57079265 0.00000735 1.57079265" />
       <geometry>
-        <mesh filename="package://adam_urdf/meshes/pe_tornozelo.STL" />
+        <mesh filename="package://adam_description/meshes/pe_tornozelo.STL" />
       </geometry>
     </collision>
@@ -151,5 +151,5 @@
       <origin xyz="-0.20764875 -0.05165039 0.02455327" rpy="-0.78539449 -1.57079113 0.78539816" />
       <geometry>
-        <mesh filename="package://adam_urdf/meshes/pe_pe.STL" />
+        <mesh filename="package://adam_description/meshes/pe_pe.STL" />
       </geometry>
       <material name="">
@@ -160,5 +160,5 @@
       <origin xyz="-0.20764875 -0.05165039 0.02455327" rpy="-0.78539449 -1.57079113 0.78539816" />
       <geometry>
-        <mesh filename="package://adam_urdf/meshes/pe_pe.STL" />
+        <mesh filename="package://adam_description/meshes/pe_pe.STL" />
       </geometry>
     </collision>
@@ -180,5 +180,5 @@
       <origin xyz="0.03625008 0.01049992 -0.02299991" rpy="2.35619449 -1.57079113 2.35619449" />
       <geometry>
-        <mesh filename="package://adam_urdf/meshes/pd_quadril.STL" />
+        <mesh filename="package://adam_description/meshes/pd_quadril.STL" />
       </geometry>
       <material name="">
@@ -189,5 +189,5 @@
       <origin xyz="0.03625008 0.01049992 -0.02299991" rpy="2.35619449 -1.57079113 2.35619449" />
       <geometry>
-        <mesh filename="package://adam_urdf/meshes/pd_quadril.STL" />
+        <mesh filename="package://adam_description/meshes/pd_quadril.STL" />
       </geometry>
     </collision>
@@ -209,5 +209,5 @@
       <origin xyz="0.05790780 -0.00175479 0.03045030" rpy="1.57079265 0.00000735 1.57079265" />
       <geometry>
-        <mesh filename="package://adam_urdf/meshes/pd_coxa.STL" />
+        <mesh filename="package://adam_description/meshes/pd_coxa.STL" />
       </geometry>
       <material name="">
@@ -218,5 +218,5 @@
       <origin xyz="0.05790780 -0.00175479 0.03045030" rpy="1.57079265 0.00000735 1.57079265" />
       <geometry>
-        <mesh filename="package://adam_urdf/meshes/pd_coxa.STL" />
+        <mesh filename="package://adam_description/meshes/pd_coxa.STL" />
       </geometry>
     </collision>
@@ -238,5 +238,5 @@
       <origin xyz="-0.01394569 0.13230775 0.03045030" rpy="1.57079265 0.00000735 3.14159265" />
       <geometry>
-        <mesh filename="package://adam_urdf/meshes/pd_canela.STL" />
+        <mesh filename="package://adam_description/meshes/pd_canela.STL" />
       </geometry>
       <material name="">
@@ -247,5 +247,5 @@
       <origin xyz="-0.01394569 0.13230775 0.03045030" rpy="1.57079265 0.00000735 3.14159265" />
       <geometry>
-        <mesh filename="package://adam_urdf/meshes/pd_canela.STL" />
+        <mesh filename="package://adam_description/meshes/pd_canela.STL" />
       </geometry>
     </collision>
@@ -267,5 +267,5 @@
       <origin xyz="-0.20754875 -0.00075345 0.03045030" rpy="1.57079265 0.00000735 -1.57079265" />
       <geometry>
-        <mesh filename="package://adam_urdf/meshes/pd_tornozelo.STL" />
+        <mesh filename="package://adam_description/meshes/pd_tornozelo.STL" />
       </geometry>
       <material name="">
@@ -276,5 +276,5 @@
       <origin xyz="-0.20754875 -0.00075345 0.03045030" rpy="1.57079265 0.00000735 -1.57079265" />
       <geometry>
-        <mesh filename="package://adam_urdf/meshes/pd_tornozelo.STL" />
+        <mesh filename="package://adam_description/meshes/pd_tornozelo.STL" />
       </geometry>
     </collision>
@@ -296,5 +296,5 @@
       <origin xyz="-0.20764875 0.05145040 0.02545327" rpy="0.78539449 -1.57079113 -0.78539816" />
       <geometry>
-        <mesh filename="package://adam_urdf/meshes/pd_pe.STL" />
+        <mesh filename="package://adam_description/meshes/pd_pe.STL" />
       </geometry>
       <material name="">
@@ -305,5 +305,5 @@
       <origin xyz="-0.20764875 0.05145040 0.02545327" rpy="0.78539449 -1.57079113 -0.78539816" />
       <geometry>
-        <mesh filename="package://adam_urdf/meshes/pd_pe.STL" />
+        <mesh filename="package://adam_description/meshes/pd_pe.STL" />
       </geometry>
     </collision>
@@ -325,5 +325,5 @@
       <origin xyz="-0.17620805 0.00549938 -0.08799998" rpy="1.57079647 -0.00000367 1.53300000" />
       <geometry>
-        <mesh filename="package://adam_urdf/meshes/be_ombro.STL" />
+        <mesh filename="package://adam_description/meshes/be_ombro.STL" />
       </geometry>
       <material name="">
@@ -334,5 +334,5 @@
       <origin xyz="-0.17620805 0.00549938 -0.08799998" rpy="1.57079647 -0.00000367 1.53300000" />
       <geometry>
-        <mesh filename="package://adam_urdf/meshes/be_ombro.STL" />
+        <mesh filename="package://adam_description/meshes/be_ombro.STL" />
       </geometry>
     </collision>
@@ -354,5 +354,5 @@
       <origin xyz="-0.15828976 0.11100006 -0.02216938" rpy="-0.19251951 -1.57075794 -2.94907300" />
       <geometry>
-        <mesh filename="package://adam_urdf/meshes/be_biceps.STL" />
+        <mesh filename="package://adam_description/meshes/be_biceps.STL" />
       </geometry>
       <material name="">
@@ -363,5 +363,5 @@
       <origin xyz="-0.15828976 0.11100006 -0.02216938" rpy="-0.19251951 -1.57075794 -2.94907300" />
       <geometry>
-        <mesh filename="package://adam_urdf/meshes/be_biceps.STL" />
+        <mesh filename="package://adam_description/meshes/be_biceps.STL" />
       </geometry>
     </collision>
@@ -383,5 +383,5 @@
       <origin xyz="-0.01936902 0.09838934 -0.13200042" rpy="1.57079279 -0.00000734 0.00003400" />
       <geometry>
-        <mesh filename="package://adam_urdf/meshes/be_antibraco.STL" />
+        <mesh filename="package://adam_description/meshes/be_antibraco.STL" />
       </geometry>
       <material name="">
@@ -392,5 +392,5 @@
       <origin xyz="-0.01936902 0.09838934 -0.13200042" rpy="1.57079279 -0.00000734 0.00003400" />
       <geometry>
-        <mesh filename="package://adam_urdf/meshes/be_antibraco.STL" />
+        <mesh filename="package://adam_description/meshes/be_antibraco.STL" />
       </geometry>
     </collision>
@@ -412,5 +412,5 @@
       <origin xyz="-0.17620805 -0.00549938 -0.08799998" rpy="-1.57079647 -0.00000367 -1.53300000" />
       <geometry>
-        <mesh filename="package://adam_urdf/meshes/bd_ombro.STL" />
+        <mesh filename="package://adam_description/meshes/bd_ombro.STL" />
       </geometry>
       <material name="">
@@ -421,5 +421,5 @@
       <origin xyz="-0.17620805 -0.00549938 -0.08799998" rpy="-1.57079647 -0.00000367 -1.53300000" />
       <geometry>
-        <mesh filename="package://adam_urdf/meshes/bd_ombro.STL" />
+        <mesh filename="package://adam_description/meshes/bd_ombro.STL" />
       </geometry>
     </collision>
@@ -441,5 +441,5 @@
       <origin xyz="-0.15828976 -0.11100006 -0.02216938" rpy="0.19251951 -1.57075794 2.94907300" />
       <geometry>
-        <mesh filename="package://adam_urdf/meshes/bd_biceps.STL" />
+        <mesh filename="package://adam_description/meshes/bd_biceps.STL" />
       </geometry>
       <material name="">
@@ -450,5 +450,5 @@
       <origin xyz="-0.15828976 -0.11100006 -0.02216938" rpy="0.19251951 -1.57075794 2.94907300" />
       <geometry>
-        <mesh filename="package://adam_urdf/meshes/bd_biceps.STL" />
+        <mesh filename="package://adam_description/meshes/bd_biceps.STL" />
       </geometry>
     </collision>
@@ -470,5 +470,5 @@
       <origin xyz="-0.01936974 -0.09839022 -0.13199967" rpy="-1.57080049 -0.00000734 -0.00004135" />
       <geometry>
-        <mesh filename="package://adam_urdf/meshes/bd_antibraco.STL" />
+        <mesh filename="package://adam_description/meshes/bd_antibraco.STL" />
       </geometry>
       <material name="">
@@ -479,5 +479,5 @@
       <origin xyz="-0.01936974 -0.09839022 -0.13199967" rpy="-1.57080049 -0.00000734 -0.00004135" />
       <geometry>
-        <mesh filename="package://adam_urdf/meshes/bd_antibraco.STL" />
+        <mesh filename="package://adam_description/meshes/bd_antibraco.STL" />
       </geometry>
     </collision>

File: src/adam_description/urdf/adam_fixed.urdf (robot description, URDF)
Before this commit: robot adam, 17 links, 16 joints
Links:
- link base_link: geometry collision mesh filename=package://adam_description/meshes/base_link.STL; visual mesh filename=package://adam_description/meshes/base_link.STL
- link bd_antibraco: geometry collision mesh filename=package://adam_description/meshes/bd_antibraco.STL; visual mesh filename=package://adam_description/meshes/bd_antibraco.STL
- link bd_biceps: geometry collision mesh filename=package://adam_description/meshes/bd_biceps.STL; visual mesh filename=package://adam_description/meshes/bd_biceps.STL
- link bd_ombro: geometry collision mesh filename=package://adam_description/meshes/bd_ombro.STL; visual mesh filename=package://adam_description/meshes/bd_ombro.STL
- link be_antibraco: geometry collision mesh filename=package://adam_description/meshes/be_antibraco.STL; visual mesh filename=package://adam_description/meshes/be_antibraco.STL
- link be_biceps: geometry collision mesh filename=package://adam_description/meshes/be_biceps.STL; visual mesh filename=package://adam_description/meshes/be_biceps.STL
- link be_ombro: geometry collision mesh filename=package://adam_description/meshes/be_ombro.STL; visual mesh filename=package://adam_description/meshes/be_ombro.STL
- link pd_canela: geometry collision mesh filename=package://adam_description/meshes/pd_canela.STL; visual mesh filename=package://adam_description/meshes/pd_canela.STL
- link pd_coxa: geometry collision mesh filename=package://adam_description/meshes/pd_coxa.STL; visual mesh filename=package://adam_description/meshes/pd_coxa.STL
- link pd_pe: geometry collision mesh filename=package://adam_description/meshes/pd_pe.STL; visual mesh filename=package://adam_description/meshes/pd_pe.STL
- link pd_quadril: geometry collision mesh filename=package://adam_description/meshes/pd_quadril.STL; visual mesh filename=package://adam_description/meshes/pd_quadril.STL
- link pd_tornozelo: geometry collision mesh filename=package://adam_description/meshes/pd_tornozelo.STL; visual mesh filename=package://adam_description/meshes/pd_tornozelo.STL
- link pe_canela: geometry collision mesh filename=package://adam_description/meshes/pe_canela.STL; visual mesh filename=package://adam_description/meshes/pe_canela.STL
- link pe_coxa: geometry collision mesh filename=package://adam_description/meshes/pe_coxa.STL; visual mesh filename=package://adam_description/meshes/pe_coxa.STL
- link pe_pe: geometry collision mesh filename=package://adam_description/meshes/pe_pe.STL; visual mesh filename=package://adam_description/meshes/pe_pe.STL
- link pe_quadril: geometry collision mesh filename=package://adam_description/meshes/pe_quadril.STL; visual mesh filename=package://adam_description/meshes/pe_quadril.STL
- link pe_tornozelo: geometry collision mesh filename=package://adam_description/meshes/pe_tornozelo.STL; visual mesh filename=package://adam_description/meshes/pe_tornozelo.STL
